File: Hardware/6502/6502-Controller.kicad_pcb (KiCad board)
At the start: 2 copper layers, 150.5 x 75.1 mm, 47 parts, among them J1 User Port One, J10 5V, J20 Switch, J21 Reset, J22 LED, J3 Expanstion Port, J4 Expansion IRQ Enable, J5 6522 IRQ Enable, J6 SERIAL IRQ Enale, J7 SERIAL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

Commit message: Update
Update of Projects
Routing:
- net (no net): track 0.00 -> 8.96 mm
Changed lines of the file:
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@@
     (thickness 1.6)
     (drawings 103)
-    (tracks 1832)
+    (tracks 1837)
     (zones 0)
     (modules 47)
@@
   (page A4)
   (layers
-    (0 F.Cu signal)
-    (31 B.Cu signal)
+    (0 F.Cu signal hide)
+    (31 B.Cu signal hide)
     (32 B.Adhes user)
     (33 F.Adhes user)
@@
     (arrow2b (pts (xy 83.566 139.319) (xy 84.692504 138.732579)))
   )
+  (segment (start 168.529 44.057) (end 169.3552 43.2308) (width 0.4) (layer B.Cu) (net 0))
+  (segment (start 168.529 45.657) (end 168.529 44.057) (width 0.4) (layer B.Cu) (net 0))
+  (segment (start 173.609 44.057) (end 173.609 45.657) (width 0.4) (layer B.Cu) (net 0))
+  (segment (start 172.7828 43.2308) (end 173.609 44.057) (width 0.4) (layer B.Cu) (net 0))
+  (segment (start 169.3552 43.2308) (end 172.7828 43.2308) (width 0.4) (layer B.Cu) (net 0))
   (segment (start 92.757 75.946) (end 93.8399 77.0289) (width 0.35) (layer B.Cu) (net 1))
   (segment (start 93.8399 77.0289) (end 93.8399 98.6241) (width 0.35) (layer B.Cu) (net 1))
